Commit message: [fix] wheelジョイントが動くように変更。

File: fourth_robot/fourth_robot_description/urdf/fourth_robot.urdf (robot description, URDF)
Before this commit: robot kit_c4, 10 links, 9 joints
Joints:
- joint base_link_to_left_wheel: origin xyz=0 0.214375 0 rpy=3.141592 0 0 -> xyz=0 0.214375 0 rpy=0 0 3.141592; type fixed -> continuous
- joint base_link_to_right_wheel: type fixed -> continuous
