Commit message: [modify] 前後マクロを削除

File: third_robot/third_robot_description/urdf/third_robot_macro.xacro (robot description, xacro)
@@ -19,4 +19,5 @@
         </inertial>
     </xacro:macro>
+    <!-- wheel macro -->
     <xacro:macro name="wheel" params="right_left reflect_right_left front_rear reflect_front_rear">
         <link name="${right_left}_${front_rear}_wheel">
@@ -45,52 +46,3 @@
         </joint>
     </xacro:macro>
-    <xacro:macro name="wheel_front" params="right_left reflect_right_left">
-        <link name="${right_left}_front_wheel">
-            <visual>
-                <!-- when reflect_right_left = 1 to be 0 reflect_right_left= -1 to be PI -->
-                <origin rpy="${PI/2-reflect_right_left*PI/2} 0 0" xyz="0 0 0"/>
-                <!-- <origin rpy="${PI/2-reflect_right_left*PI/2} 0 0" xyz="0 0 0"/> -->
-                <geometry>
-                    <mesh filename="package://third_robot_description/meshes/third_robot/third_robot_wheel.dae"/>
-                </geometry>
-                ->
-            </visual>
-            <collision>
-                <origin rpy="${PI/2} 0 0" xyz="0 0 0"/>
-                <geometry>
-                    <cylinder length="${length_wheel}" radius="${radius_wheel}"/>
-                </geometry>
-            </collision>
-            <xacro:default_inertial mass="1"/>
-        </link>
-        <joint name="base_to_${right_left}_front_wheel" type="continuous">
-            <axis xyz="0 1 0"/>
-            <parent link="base_link"/>
-            <child link="${right_left}_front_wheel"/>
-            <origin xyz="${base_center_x+length_from_base_center_to_wheel_x} ${-reflect_right_left*length_from_base_to_wheel_y} ${radius_wheel}"/>
-        </joint>
-    </xacro:macro>
-    <xacro:macro name="wheel_rear" params="right_left reflect_right_left">
-        <link name="${right_left}_rear_wheel">
-            <visual>
-                <origin rpy="${PI/2-reflect_right_left*PI/2} 0 0" xyz="0 0 0"/>
-                <geometry>
-                    <mesh filename="package://third_robot_description/meshes/third_robot/third_robot_wheel.dae"/>
-                </geometry>
-            </visual>
-            <collision>
-                <origin rpy="${PI/2} 0 0" xyz="0 0 0"/>
-                <geometry>
-                    <cylinder length="${length_wheel}" radius="${radius_wheel}"/>
-                </geometry>
-            </collision>
-            <xacro:default_inertial mass="1"/>
-        </link>
-        <joint name="base_to_${right_left}_rear_wheel" type="continuous">
-            <axis xyz="0 1 0"/>
-            <parent link="base_link"/>
-            <child link="${right_left}_rear_wheel"/>
-            <origin xyz="${base_center_x-length_from_base_center_to_wheel_x} ${-reflect_right_left*length_from_base_to_wheel_y} ${radius_wheel}"/>
-        </joint>
-    </xacro:macro>
 </robot>
