Commit message: [fix] LRFの角度とかrvizのコンフィグを追加。

File: third_robot/third_robot_description/urdf/third_robot.urdf (robot description, URDF)
Before this commit: robot origins, 8 links, 7 joints
Joints:
- joint base_to_front_top_lrf: origin xyz=0.40 0 0.75 -> xyz=0.40 0 0.75 rpy=0 0.57 0

Commit message: [fix] 実験的なパラメータ調整など

File: third_robot/third_robot_description/urdf/third_robot.urdf (robot description, URDF)
Before this commit: robot origins, 8 links, 7 joints
Joints:
- joint base_to_front_top_lrf: origin xyz=0.40 0 0.75 rpy=0 0.57 0 -> xyz=0.40 0 0.75 rpy=0 0.53 0

Commit message: [fix] base_linkの位置を変更した。

File: third_robot/third_robot_description/urdf/third_robot.urdf (robot description, URDF)
Before this commit: robot origins, 8 links, 7 joints
Joints:
- joint base_to_front_bottom_lrf: origin xyz=0.50 0 0.39 -> xyz=0.88 0 0.39
- joint base_to_front_top_lrf: origin xyz=0.40 0 0.75 rpy=0 0.53 0 -> xyz=0.78 0 0.75 rpy=0 0.53 0
- joint base_to_left_front_wheel: origin xyz=0.41 0.25 0.14 -> xyz=0.79 0.25 0.14
- joint base_to_left_rear_wheel: origin xyz=-0.38 0.25 0.14 -> xyz=0 0.25 0.14
- joint base_to_rear_bottom_lrf: origin xyz=-0.45 0 0.35 -> xyz=-0.07 0 0.35
- joint base_to_right_front_wheel: origin xyz=0.41 -0.25 0.14 -> xyz=0.79 -0.25 0.14
- joint base_to_right_rear_wheel: origin xyz=-0.38 -0.25 0.14 -> xyz=0 -0.25 0.14

Commit message: [modify] 後ろのLRFの位置を修正

File: third_robot/third_robot_description/urdf/third_robot.urdf (robot description, URDF)
Before this commit: robot origins, 8 links, 7 joints
Joints:
- joint base_to_rear_bottom_lrf: origin xyz=-0.07 0 0.35 -> xyz=-0.07 0 0.39

Commit message: [fix] いろいろ修正

File: third_robot/third_robot_description/urdf/third_robot.urdf (robot description, URDF)
Before this commit: robot origins, 8 links, 7 joints
Joints:
- joint base_to_rear_bottom_lrf: origin xyz=-0.07 0 0.39 -> xyz=-0.07 0 0.39 rpy=0 0 3.1416

Commit message: [fix] いろいろ修正

File: third_robot/third_robot_description/urdf/third_robot.urdf (robot description, URDF)
Before this commit: robot origins, 8 links, 7 joints
Links:
- added link merged_lrf
Joints:
- added joint base_to_merged_lrf: type fixed, parent base_link, child merged_lrf, origin xyz=0 0 0.39 rpy=0 0 0, axis 0 1 0

Commit message: Revert "Modify third robot driver"

File: third_robot/third_robot_description/urdf/third_robot.urdf (robot description, URDF)
Before this commit: robot origins, 9 links, 8 joints
Links:
- removed link merged_lrf
Joints:
- removed joint base_to_merged_lrf
- joint base_to_rear_bottom_lrf: origin xyz=-0.07 0 0.39 rpy=0 0 3.1416 -> xyz=-0.07 0 0.35
