Commit message: [add] 独立二輪を想定したシミュレーションモデルで車輪が動くとこまで2

File: third_robot/third_robot_description/urdf/third_robot.xacro (robot description, xacro)
@@ -97,5 +97,5 @@
         <collision>
             <geometry>
-                <cylinder length="${length_wheel}" radius="${radius_wheel}"/>
+                <cylinder length="${length_wheel}" radius="${radius_wheel}25"/>
             </geometry>
         </collision>
@@ -150,3 +150,23 @@
         <origin xyz="-0.45 0 0.35"/>
     </joint>
+    <transmission name="tran1">
+        <type>transmission_interface/SimpleTransmission</type>
+        <joint name="base_to_left_rear_wheel">
+            <hardwareInterface>EffortJointInterface</hardwareInterface>
+        </joint>
+        <actuator name="motor1">
+            <hardwareInterface>EffortJointInterface</hardwareInterface>
+            <mechanicalReduction>1</mechanicalReduction>
+        </actuator>
+    </transmission>
+    <transmission name="tran2">
+        <type>transmission_interface/SimpleTransmission</type>
+        <joint name="base_to_right_rear_wheel">
+            <hardwareInterface>EffortJointInterface</hardwareInterface>
+        </joint>
+        <actuator name="motor2">
+            <hardwareInterface>EffortJointInterface</hardwareInterface>
+            <mechanicalReduction>1</mechanicalReduction>
+        </actuator>
+    </transmission>
 </robot>

Commit message: [add] 走るけど多分車輪軸ずれている

File: third_robot/third_robot_description/urdf/third_robot.xacro (robot description, xacro)
@@ -23,5 +23,5 @@
         <collision>
             <geometry>
-                <box size="1.5 1.5 0.005"/>
+                <box size="0.5 1.5 0.0"/>
             </geometry>
         </collision>
@@ -97,5 +97,5 @@
         <collision>
             <geometry>
-                <cylinder length="${length_wheel}" radius="${radius_wheel}25"/>
+                <cylinder length="${length_wheel}" radius="${radius_wheel}"/>
             </geometry>
         </collision>

Commit message: [modify] 3号機前進！

File: third_robot/third_robot_description/urdf/third_robot.xacro (robot description, xacro)
@@ -3,10 +3,12 @@
     <!-- Import all Gazebo-customization elements, including Gazebo colors -->
     <xacro:include filename="$(find third_robot_description)/urdf/third_robot.gazebo" />
+    <!-- Constants for math -->
+    <xacro:property name="PI" value="3.1415926535897931" />
     <!-- Constants for robot dimensions -->
-    <xacro:property name="length_wheel" value="0.05" />
-    <xacro:property name="radius_wheel" value="0.12" />
+    <xacro:property name="length_wheel" value="0.07" />
+    <xacro:property name="radius_wheel" value="0.14" />
     <xacro:macro name="default_inertial" params="mass">
         <inertial>
-            <mass value="${mass}" />
+            ,05<mass value="${mass}" />
             <inertia ixx="1.0" ixy="0.0" ixz="0.0"
                 iyy="1.0" iyz="0.0"
@@ -18,4 +20,5 @@
             <geometry>
                 <mesh filename="package://third_robot_description/meshes/third_robot/third_robot_body.dae"/>
+                <box size="1.05 0.55 0.6"/>
             </geometry>
             <origin rpy="0 0 0" xyz="0 0 0.55" />
@@ -31,9 +34,16 @@
         <visual>
             <geometry>
+                <!--
                 <mesh filename="package://third_robot_description/meshes/third_robot/third_robot_wheel.dae"/>
+                -->
+                <cylinder length="${length_wheel}" radius="${radius_wheel}"/>
             </geometry>
+            <origin rpy="${3.14159/2} 0 0" xyz="0 0 0"/>
+                <!--
             <origin rpy="0 0 0" xyz="0 0 0"/>
+                -->
         </visual>
         <collision>
+            <origin rpy="${3.14159/2} 0 0" xyz="0 0 0"/>
             <geometry>
                 <cylinder length="${length_wheel}" radius="${radius_wheel}"/>
@@ -53,7 +63,8 @@
                 <mesh filename="package://third_robot_description/meshes/third_robot/third_robot_wheel.dae"/>
             </geometry>
-            <origin rpy="3.14159 0 0" xyz="0 0 0"/>
+            <origin rpy="${PI} 0 0" xyz="0 0 0"/>
         </visual>
         <collision>
+            <origin rpy="${PI/2} 0 0" xyz="0 0 0"/>
             <geometry>
                 <cylinder length="${length_wheel}" radius="${radius_wheel}"/>
@@ -76,4 +87,5 @@
         </visual>
         <collision>
+            <origin rpy="${3.14159/2} 0 0" xyz="0 0 0"/>
             <geometry>
                 <cylinder length="${length_wheel}" radius="${radius_wheel}"/>
@@ -96,4 +108,5 @@
         </visual>
         <collision>
+            <origin rpy="${3.14159/2} 0 0" xyz="0 0 0"/>
             <geometry>
                 <cylinder length="${length_wheel}" radius="${radius_wheel}"/>

Commit message: [modify] 車輪の半径を修正

File: third_robot/third_robot_description/urdf/third_robot.xacro (robot description, xacro)
@@ -10,5 +10,5 @@
     <xacro:macro name="default_inertial" params="mass">
         <inertial>
-            ,05<mass value="${mass}" />
+            <mass value="${mass}" />
             <inertia ixx="1.0" ixy="0.0" ixz="0.0"
                 iyy="1.0" iyz="0.0"
@@ -18,13 +18,13 @@
     <link name="base_link">
         <visual>
+            <origin rpy="0 0 0" xyz="0 0 0.55" />
             <geometry>
                 <mesh filename="package://third_robot_description/meshes/third_robot/third_robot_body.dae"/>
-                <box size="1.05 0.55 0.6"/>
             </geometry>
-            <origin rpy="0 0 0" xyz="0 0 0.55" />
         </visual>
         <collision>
+            <origin rpy="0 0 0" xyz="0 0 0.35" />
             <geometry>
-                <box size="0.5 1.5 0.0"/>
+                <box size="1.05 0.55 0.4"/>
             </geometry>
         </collision>
@@ -33,17 +33,11 @@
     <link name="right_front_wheel">
         <visual>
+            <origin rpy="0 0 0" xyz="0 0 0"/>
             <geometry>
-                <!--
                 <mesh filename="package://third_robot_description/meshes/third_robot/third_robot_wheel.dae"/>
-                -->
-                <cylinder length="${length_wheel}" radius="${radius_wheel}"/>
             </geometry>
-            <origin rpy="${3.14159/2} 0 0" xyz="0 0 0"/>
-                <!--
-            <origin rpy="0 0 0" xyz="0 0 0"/>
-                -->
         </visual>
         <collision>
-            <origin rpy="${3.14159/2} 0 0" xyz="0 0 0"/>
+            <origin rpy="${PI/2} 0 0" xyz="0 0 0"/>
             <geometry>
                 <cylinder length="${length_wheel}" radius="${radius_wheel}"/>
@@ -60,8 +54,8 @@
     <link name="left_front_wheel">
         <visual>
+            <origin rpy="${PI} 0 0" xyz="0 0 0"/>
             <geometry>
                 <mesh filename="package://third_robot_description/meshes/third_robot/third_robot_wheel.dae"/>
             </geometry>
-            <origin rpy="${PI} 0 0" xyz="0 0 0"/>
         </visual>
         <collision>
@@ -81,11 +75,11 @@
     <link name="right_rear_wheel">
         <visual>
+            <origin rpy="0 0 0" xyz="0 0 0"/>
             <geometry>
                 <mesh filename="package://third_robot_description/meshes/third_robot/third_robot_wheel.dae"/>
             </geometry>
-            <origin rpy="0 0 0" xyz="0 0 0"/>
         </visual>
         <collision>
-            <origin rpy="${3.14159/2} 0 0" xyz="0 0 0"/>
+            <origin rpy="${PI/2} 0 0" xyz="0 0 0"/>
             <geometry>
                 <cylinder length="${length_wheel}" radius="${radius_wheel}"/>
@@ -102,11 +96,11 @@
     <link name="left_rear_wheel">
         <visual>
+            <origin rpy="${PI} 0 0" xyz="0 0 0"/>
             <geometry>
                 <mesh filename="package://third_robot_description/meshes/third_robot/third_robot_wheel.dae"/>
             </geometry>
-            <origin rpy="3.14159 0 0" xyz="0 0 0"/>
         </visual>
         <collision>
-            <origin rpy="${3.14159/2} 0 0" xyz="0 0 0"/>
+            <origin rpy="${PI/2} 0 0" xyz="0 0 0"/>
             <geometry>
                 <cylinder length="${length_wheel}" radius="${radius_wheel}"/>
@@ -123,8 +117,8 @@
     <link name="front_top_lrf">
         <visual>
+            <origin rpy="0 0.5 0" xyz="0 0 0"/>
             <geometry>
                 <mesh filename="package://third_robot_description/meshes/LRF/UTM-30LX.dae"/>
             </geometry>
-            <origin rpy="0 0.5 0" xyz="0 0 0"/>
         </visual>
     </link>
@@ -137,8 +131,8 @@
     <link name="front_bottom_lrf">
         <visual>
+            <origin rpy="0 0 0" xyz="0 0 0"/>
             <geometry>
                 <mesh filename="package://third_robot_description/meshes/LRF/UTM-30LX.dae"/>
             </geometry>
-            <origin rpy="0 0 0" xyz="0 0 0"/>
         </visual>
     </link>
@@ -151,8 +145,8 @@
     <link name="rear_bottom_lrf">
         <visual>
+            <origin rpy="0 0 ${PI}" xyz="0 0 0"/>
             <geometry>
                 <mesh filename="package://third_robot_description/meshes/LRF/UTM-30LX.dae"/>
             </geometry>
-            <origin rpy="0 0 3.14" xyz="0 0 0"/>
         </visual>
     </link>

Commit message: [modify] 車輪の位置を変数に集約

File: third_robot/third_robot_description/urdf/third_robot.xacro (robot description, xacro)
@@ -8,4 +8,6 @@
     <xacro:property name="length_wheel" value="0.07" />
     <xacro:property name="radius_wheel" value="0.14" />
+    <xacro:property name="length_from_base_to_wheel_front_x" value="0.41" />
+    <xacro:property name="length_from_base_to_wheel_y" value="0.25" />
     <xacro:macro name="default_inertial" params="mass">
         <inertial>
@@ -50,5 +52,5 @@
         <parent link="base_link"/>
         <child link="right_front_wheel"/>
-        <origin xyz="0.41 -0.25 0.14"/>
+        <origin xyz="${length_from_base_to_wheel_front_x} -${length_from_base_to_wheel_y} ${radius_wheel}"/>
     </joint>
     <link name="left_front_wheel">
@@ -71,5 +73,5 @@
         <parent link="base_link"/>
         <child link="left_front_wheel"/>
-        <origin xyz="0.41 0.25 0.14"/>
+        <origin xyz="${length_from_base_to_wheel_front_x} ${length_from_base_to_wheel_y} ${radius_wheel}"/>
     </joint>
     <link name="right_rear_wheel">
@@ -92,5 +94,5 @@
         <parent link="base_link"/>
         <child link="right_rear_wheel"/>
-        <origin xyz="-0.38 -0.25 0.14"/>
+        <origin xyz="-0.38 -${length_from_base_to_wheel_y} ${radius_wheel}"/>
     </joint>
     <link name="left_rear_wheel">
@@ -113,5 +115,5 @@
         <parent link="base_link"/>
         <child link="left_rear_wheel"/>
-        <origin xyz="-0.38 0.25 0.14"/>
+        <origin xyz="-0.38 ${length_from_base_to_wheel_y} ${radius_wheel}"/>
     </joint>
     <link name="front_top_lrf">
@@ -157,4 +159,5 @@
         <origin xyz="-0.45 0 0.35"/>
     </joint>
+<!--
     <transmission name="tran1">
         <type>transmission_interface/SimpleTransmission</type>
@@ -177,3 +180,4 @@
         </actuator>
     </transmission>
+-->
 </robot>

Commit message: [modify] xacro マクロ部を別ファイルに

File: third_robot/third_robot_description/urdf/third_robot.xacro (robot description, xacro)
@@ -3,19 +3,5 @@
     <!-- Import all Gazebo-customization elements, including Gazebo colors -->
     <xacro:include filename="$(find third_robot_description)/urdf/third_robot.gazebo" />
-    <!-- Constants for math -->
-    <xacro:property name="PI" value="3.1415926535897931" />
-    <!-- Constants for robot dimensions -->
-    <xacro:property name="length_wheel" value="0.07" />
-    <xacro:property name="radius_wheel" value="0.14" />
-    <xacro:property name="length_from_base_to_wheel_front_x" value="0.41" />
-    <xacro:property name="length_from_base_to_wheel_y" value="0.25" />
-    <xacro:macro name="default_inertial" params="mass">
-        <inertial>
-            <mass value="${mass}" />
-            <inertia ixx="1.0" ixy="0.0" ixz="0.0"
-                iyy="1.0" iyz="0.0"
-                izz="1.0" />
-        </inertial>
-    </xacro:macro>
+    <xacro:include filename="$(find third_robot_description)/urdf/third_robot_macro.xacro" />
     <link name="base_link">
         <visual>

Commit message: [modify] 前輪をxacroマクロ化

File: third_robot/third_robot_description/urdf/third_robot.xacro (robot description, xacro)
@@ -19,46 +19,6 @@
         <xacro:default_inertial mass="10"/>
     </link>
-    <link name="right_front_wheel">
-        <visual>
-            <origin rpy="0 0 0" xyz="0 0 0"/>
-            <geometry>
-                <mesh filename="package://third_robot_description/meshes/third_robot/third_robot_wheel.dae"/>
-            </geometry>
-        </visual>
-        <collision>
-            <origin rpy="${PI/2} 0 0" xyz="0 0 0"/>
-            <geometry>
-                <cylinder length="${length_wheel}" radius="${radius_wheel}"/>
-            </geometry>
-        </collision>
-        <xacro:default_inertial mass="1"/>
-    </link>
-    <joint name="base_to_right_front_wheel" type="continuous">
-        <axis xyz="0 1 0"/>
-        <parent link="base_link"/>
-        <child link="right_front_wheel"/>
-        <origin xyz="${length_from_base_to_wheel_front_x} -${length_from_base_to_wheel_y} ${radius_wheel}"/>
-    </joint>
-    <link name="left_front_wheel">
-        <visual>
-            <origin rpy="${PI} 0 0" xyz="0 0 0"/>
-            <geometry>
-                <mesh filename="package://third_robot_description/meshes/third_robot/third_robot_wheel.dae"/>
-            </geometry>
-        </visual>
-        <collision>
-            <origin rpy="${PI/2} 0 0" xyz="0 0 0"/>
-            <geometry>
-                <cylinder length="${length_wheel}" radius="${radius_wheel}"/>
-            </geometry>
-        </collision>
-        <xacro:default_inertial mass="1"/>
-    </link>
-    <joint name="base_to_left_front_wheel" type="continuous">
-        <axis xyz="0 1 0"/>
-        <parent link="base_link"/>
-        <child link="left_front_wheel"/>
-        <origin xyz="${length_from_base_to_wheel_front_x} ${length_from_base_to_wheel_y} ${radius_wheel}"/>
-    </joint>
+    <xacro:wheel right_left="right" reflect="1"/>
+    <xacro:wheel right_left="left" reflect="-1"/>
     <link name="right_rear_wheel">
         <visual>

File: third_robot/third_robot_description/urdf/third_robot_macro.xacro (robot description, xacro)
@@ -16,3 +16,29 @@
         </inertial>
     </xacro:macro>
+    <xacro:macro name="wheel" params="right_left reflect">
+        <link name="${right_left}_front_wheel">
+            <visual>
+                <!-- when reflect = 1 to be 0 reflect= -1 to be PI -->
+                <origin rpy="${PI/2-reflect*PI/2} 0 0" xyz="0 0 0"/>
+                <!-- <origin rpy="${PI/2-reflect*PI/2} 0 0" xyz="0 0 0"/> -->
+                <geometry>
+                    <mesh filename="package://third_robot_description/meshes/third_robot/third_robot_wheel.dae"/>
+                </geometry>
+                ->
+            </visual>
+            <collision>
+                <origin rpy="${PI/2} 0 0" xyz="0 0 0"/>
+                <geometry>
+                    <cylinder length="${length_wheel}" radius="${radius_wheel}"/>
+                </geometry>
+            </collision>
+            <xacro:default_inertial mass="1"/>
+        </link>
+        <joint name="base_to_${right_left}_front_wheel" type="continuous">
+            <axis xyz="0 1 0"/>
+            <parent link="base_link"/>
+            <child link="${right_left}_front_wheel"/>
+            <origin xyz="${length_from_base_to_wheel_front_x} ${-reflect*length_from_base_to_wheel_y} ${radius_wheel}"/>
+        </joint>
+    </xacro:macro>
 </robot>

Commit message: [modify] 後輪をxacroマクロ化

File: third_robot/third_robot_description/urdf/third_robot.xacro (robot description, xacro)
@@ -19,48 +19,8 @@
         <xacro:default_inertial mass="10"/>
     </link>
-    <xacro:wheel right_left="right" reflect="1"/>
-    <xacro:wheel right_left="left" reflect="-1"/>
-    <link name="right_rear_wheel">
-        <visual>
-            <origin rpy="0 0 0" xyz="0 0 0"/>
-            <geometry>
-                <mesh filename="package://third_robot_description/meshes/third_robot/third_robot_wheel.dae"/>
-            </geometry>
-        </visual>
-        <collision>
-            <origin rpy="${PI/2} 0 0" xyz="0 0 0"/>
-            <geometry>
-                <cylinder length="${length_wheel}" radius="${radius_wheel}"/>
-            </geometry>
-        </collision>
-        <xacro:default_inertial mass="1"/>
-    </link>
-    <joint name="base_to_right_rear_wheel" type="continuous">
-        <axis xyz="0 1 0"/>
-        <parent link="base_link"/>
-        <child link="right_rear_wheel"/>
-        <origin xyz="-0.38 -${length_from_base_to_wheel_y} ${radius_wheel}"/>
-    </joint>
-    <link name="left_rear_wheel">
-        <visual>
-            <origin rpy="${PI} 0 0" xyz="0 0 0"/>
-            <geometry>
-                <mesh filename="package://third_robot_description/meshes/third_robot/third_robot_wheel.dae"/>
-            </geometry>
-        </visual>
-        <collision>
-            <origin rpy="${PI/2} 0 0" xyz="0 0 0"/>
-            <geometry>
-                <cylinder length="${length_wheel}" radius="${radius_wheel}"/>
-            </geometry>
-        </collision>
-        <xacro:default_inertial mass="1"/>
-    </link>
-    <joint name="base_to_left_rear_wheel" type="continuous">
-        <axis xyz="0 1 0"/>
-        <parent link="base_link"/>
-        <child link="left_rear_wheel"/>
-        <origin xyz="-0.38 ${length_from_base_to_wheel_y} ${radius_wheel}"/>
-    </joint>
+    <xacro:wheel_front right_left="right" reflect="1"/>
+    <xacro:wheel_front right_left="left" reflect="-1"/>
+    <xacro:wheel_rear right_left="right" reflect="1"/>
+    <xacro:wheel_rear right_left="left" reflect="-1"/>
     <link name="front_top_lrf">
         <visual>

File: third_robot/third_robot_description/urdf/third_robot_macro.xacro (robot description, xacro)
@@ -6,5 +6,8 @@
     <xacro:property name="length_wheel" value="0.07" />
     <xacro:property name="radius_wheel" value="0.14" />
+    <xacro:property name="base_center_x" value="0.015" />
+    <xacro:property name="length_from_base_center_to_wheel_x" value="0.395" />
     <xacro:property name="length_from_base_to_wheel_front_x" value="0.41" />
+    <xacro:property name="length_from_base_to_wheel_rear_x" value="0.38" />
     <xacro:property name="length_from_base_to_wheel_y" value="0.25" />
     <xacro:macro name="default_inertial" params="mass">
@@ -16,5 +19,5 @@
         </inertial>
     </xacro:macro>
-    <xacro:macro name="wheel" params="right_left reflect">
+    <xacro:macro name="wheel_front" params="right_left reflect">
         <link name="${right_left}_front_wheel">
             <visual>
@@ -39,5 +42,28 @@
             <parent link="base_link"/>
             <child link="${right_left}_front_wheel"/>
-            <origin xyz="${length_from_base_to_wheel_front_x} ${-reflect*length_from_base_to_wheel_y} ${radius_wheel}"/>
+            <origin xyz="${base_center_x+length_from_base_center_to_wheel_x} ${-reflect*length_from_base_to_wheel_y} ${radius_wheel}"/>
+        </joint>
+    </xacro:macro>
+    <xacro:macro name="wheel_rear" params="right_left reflect">
+        <link name="${right_left}_rear_wheel">
+            <visual>
+                <origin rpy="${PI/2-reflect*PI/2} 0 0" xyz="0 0 0"/>
+                <geometry>
+                    <mesh filename="package://third_robot_description/meshes/third_robot/third_robot_wheel.dae"/>
+                </geometry>
+            </visual>
+            <collision>
+                <origin rpy="${PI/2} 0 0" xyz="0 0 0"/>
+                <geometry>
+                    <cylinder length="${length_wheel}" radius="${radius_wheel}"/>
+                </geometry>
+            </collision>
+            <xacro:default_inertial mass="1"/>
+        </link>
+        <joint name="base_to_${right_left}_rear_wheel" type="continuous">
+            <axis xyz="0 1 0"/>
+            <parent link="base_link"/>
+            <child link="${right_left}_rear_wheel"/>
+            <origin xyz="${base_center_x-length_from_base_center_to_wheel_x} ${-reflect*length_from_base_to_wheel_y} ${radius_wheel}"/>
         </joint>
     </xacro:macro>
