Commit message: [modify] 前後、左右共に引数で指定できるよう準備

File: third_robot/third_robot_description/urdf/third_robot.xacro (robot description, xacro)
@@ -19,8 +19,8 @@
         <xacro:default_inertial mass="10"/>
     </link>
-    <xacro:wheel_front right_left="right" reflect="1"/>
-    <xacro:wheel_front right_left="left" reflect="-1"/>
-    <xacro:wheel_rear right_left="right" reflect="1"/>
-    <xacro:wheel_rear right_left="left" reflect="-1"/>
+    <xacro:wheel_front right_left="right" reflect_right_left="1"/>
+    <xacro:wheel_front right_left="left" reflect_right_left="-1"/>
+    <xacro:wheel_rear right_left="right" reflect_right_left="1"/>
+    <xacro:wheel_rear right_left="left" reflect_right_left="-1"/>
     <link name="front_top_lrf">
         <visual>

File: third_robot/third_robot_description/urdf/third_robot_macro.xacro (robot description, xacro)
@@ -19,10 +19,10 @@
         </inertial>
     </xacro:macro>
-    <xacro:macro name="wheel_front" params="right_left reflect">
+    <xacro:macro name="wheel_front" params="right_left reflect_right_left">
         <link name="${right_left}_front_wheel">
             <visual>
-                <!-- when reflect = 1 to be 0 reflect= -1 to be PI -->
-                <origin rpy="${PI/2-reflect*PI/2} 0 0" xyz="0 0 0"/>
-                <!-- <origin rpy="${PI/2-reflect*PI/2} 0 0" xyz="0 0 0"/> -->
+                <!-- when reflect_right_left = 1 to be 0 reflect_right_left= -1 to be PI -->
+                <origin rpy="${PI/2-reflect_right_left*PI/2} 0 0" xyz="0 0 0"/>
+                <!-- <origin rpy="${PI/2-reflect_right_left*PI/2} 0 0" xyz="0 0 0"/> -->
                 <geometry>
                     <mesh filename="package://third_robot_description/meshes/third_robot/third_robot_wheel.dae"/>
@@ -42,11 +42,11 @@
             <parent link="base_link"/>
             <child link="${right_left}_front_wheel"/>
-            <origin xyz="${base_center_x+length_from_base_center_to_wheel_x} ${-reflect*length_from_base_to_wheel_y} ${radius_wheel}"/>
+            <origin xyz="${base_center_x+length_from_base_center_to_wheel_x} ${-reflect_right_left*length_from_base_to_wheel_y} ${radius_wheel}"/>
         </joint>
     </xacro:macro>
-    <xacro:macro name="wheel_rear" params="right_left reflect">
+    <xacro:macro name="wheel_rear" params="right_left reflect_right_left">
         <link name="${right_left}_rear_wheel">
             <visual>
-                <origin rpy="${PI/2-reflect*PI/2} 0 0" xyz="0 0 0"/>
+                <origin rpy="${PI/2-reflect_right_left*PI/2} 0 0" xyz="0 0 0"/>
                 <geometry>
                     <mesh filename="package://third_robot_description/meshes/third_robot/third_robot_wheel.dae"/>
@@ -65,5 +65,5 @@
             <parent link="base_link"/>
             <child link="${right_left}_rear_wheel"/>
-            <origin xyz="${base_center_x-length_from_base_center_to_wheel_x} ${-reflect*length_from_base_to_wheel_y} ${radius_wheel}"/>
+            <origin xyz="${base_center_x-length_from_base_center_to_wheel_x} ${-reflect_right_left*length_from_base_to_wheel_y} ${radius_wheel}"/>
         </joint>
     </xacro:macro>

Commit message: [modify] 前後左右マクロを1つに集約

File: third_robot/third_robot_description/urdf/third_robot.xacro (robot description, xacro)
@@ -19,8 +19,10 @@
         <xacro:default_inertial mass="10"/>
     </link>
-    <xacro:wheel_front right_left="right" reflect_right_left="1"/>
-    <xacro:wheel_front right_left="left" reflect_right_left="-1"/>
-    <xacro:wheel_rear right_left="right" reflect_right_left="1"/>
-    <xacro:wheel_rear right_left="left" reflect_right_left="-1"/>
+    <!-- wheels -->
+    <xacro:wheel right_left="right" reflect_right_left="1" front_rear="front" reflect_front_rear="1"/>
+    <xacro:wheel right_left="left" reflect_right_left="-1" front_rear="front" reflect_front_rear="1"/>
+    <xacro:wheel right_left="right" reflect_right_left="1" front_rear="rear" reflect_front_rear="-1"/>
+    <xacro:wheel right_left="left" reflect_right_left="-1" front_rear="rear" reflect_front_rear="-1"/>
+    <!-- lrf -->
     <link name="front_top_lrf">
         <visual>

File: third_robot/third_robot_description/urdf/third_robot_macro.xacro (robot description, xacro)
@@ -18,4 +18,30 @@
                 izz="1.0" />
         </inertial>
+    </xacro:macro>
+    <xacro:macro name="wheel" params="right_left reflect_right_left front_rear reflect_front_rear">
+        <link name="${right_left}_${front_rear}_wheel">
+            <visual>
+                <!-- when reflect_right_left = 1 to be 0 reflect_right_left= -1 to be PI -->
+                <origin rpy="${PI/2-reflect_right_left*PI/2} 0 0" xyz="0 0 0"/>
+                <!-- <origin rpy="${PI/2-reflect_right_left*PI/2} 0 0" xyz="0 0 0"/> -->
+                <geometry>
+                    <mesh filename="package://third_robot_description/meshes/third_robot/third_robot_wheel.dae"/>
+                </geometry>
+                ->
+            </visual>
+            <collision>
+                <origin rpy="${PI/2} 0 0" xyz="0 0 0"/>
+                <geometry>
+                    <cylinder length="${length_wheel}" radius="${radius_wheel}"/>
+                </geometry>
+            </collision>
+            <xacro:default_inertial mass="1"/>
+        </link>
+        <joint name="base_to_${right_left}_${front_rear}_wheel" type="continuous">
+            <axis xyz="0 1 0"/>
+            <parent link="base_link"/>
+            <child link="${right_left}_${front_rear}_wheel"/>
+            <origin xyz="${base_center_x+reflect_front_rear*length_from_base_center_to_wheel_x} ${-reflect_right_left*length_from_base_to_wheel_y} ${radius_wheel}"/>
+        </joint>
     </xacro:macro>
     <xacro:macro name="wheel_front" params="right_left reflect_right_left">

Commit message: [add] 正面カメラ追加

File: third_robot/third_robot_description/urdf/third_robot.xacro (robot description, xacro)
@@ -1,6 +1,10 @@
 <?xml version="1.0"?>
 <robot name="origins" xmlns:xacro="http://www.ros.org/wiki/xacro">
+    <xacro:property name="camera_link" value="0.05" /> <!-- Size of square 'camera' box -->
     <!-- Import all Gazebo-customization elements, including Gazebo colors -->
     <xacro:include filename="$(find third_robot_description)/urdf/third_robot.gazebo" />
+    <!-- Import Rviz colors -->
+    <xacro:include filename="$(find third_robot_description)/urdf/materials.xacro" />
+    <!-- Import macros -->
     <xacro:include filename="$(find third_robot_description)/urdf/third_robot_macro.xacro" />
     <link name="base_link">
@@ -14,5 +18,5 @@
             <origin rpy="0 0 0" xyz="0 0 0.35" />
             <geometry>
-                <box size="1.05 0.55 0.4"/>
+                <box size="1.0 0.55 0.4"/>
             </geometry>
         </collision>
@@ -67,4 +71,31 @@
         <origin xyz="-0.45 0 0.35"/>
     </joint>
+    <!-- Camera -->
+    <link name="camera_link">
+        <collision>
+            <origin xyz="0 0 0" rpy="0 0 0"/>
+            <geometry>
+                <box size="${camera_link/3} ${camera_link} ${camera_link/2}"/>
+            </geometry>
+        </collision>
+        <visual>
+            <origin xyz="0 0 0" rpy="0 0 0"/>
+            <geometry>
+                <box size="${camera_link/3} ${camera_link} ${camera_link/2}"/>
+            </geometry>
+            <material name="black"/>
+        </visual>
+        <inertial>
+            <mass value="1e-5" />
+            <origin xyz="0 0 0" rpy="0 0 0"/>
+            <inertia ixx="1e-6" ixy="0" ixz="0" iyy="1e-6" iyz="0" izz="1e-6" />
+        </inertial>
+    </link>
+    <joint name="base_to_camera" type="fixed">
+        <axis xyz="0 1 0" />
+        <parent link="base_link"/>
+        <child link="camera_link"/>
+        <origin rpy="0 0 0" xyz="0.45 0 0.72"/>
+    </joint>
 <!--
     <transmission name="tran1">

Commit message: [fix] ホイールのフレームが出るようtransmissionタグを追加

File: third_robot/third_robot_description/urdf/third_robot.xacro (robot description, xacro)
@@ -98,5 +98,4 @@
         <origin rpy="0 0 0" xyz="0.45 0 0.72"/>
     </joint>
-<!--
     <transmission name="tran1">
         <type>transmission_interface/SimpleTransmission</type>
@@ -119,4 +118,3 @@
         </actuator>
     </transmission>
--->
 </robot>

File: third_robot/third_robot_description/urdf/third_robot_macro.xacro (robot description, xacro)
@@ -45,4 +45,14 @@
             <origin xyz="${base_center_x+reflect_front_rear*length_from_base_center_to_wheel_x} ${-reflect_right_left*length_from_base_to_wheel_y} ${radius_wheel}"/>
         </joint>
+        <transmission name="tran_${right_left}_${front_rear}">
+            <type>transmission_interface/SimpleTransmission</type>
+            <joint name="base_to_${right_left}_${front_rear}_wheel">
+                <hardwareInterface>EffortJointInterface</hardwareInterface>
+            </joint>
+            <actuator name="${right_left}_${front_rear}">
+                <hardwareInterface>EffortJointInterface</hardwareInterface>
+                <mechanicalReduction>1</mechanicalReduction>
+            </actuator>
+        </transmission>
     </xacro:macro>
 </robot>

Commit message: [add] 後方LRF追加。

File: third_robot/third_robot_description/urdf/third_robot.xacro (robot description, xacro)
@@ -69,5 +69,5 @@
         <parent link="base_link"/>
         <child link="rear_bottom_lrf"/>
-        <origin xyz="-0.45 0 0.35"/>
+        <origin  rpy="0 0 ${PI}" xyz="-0.45 0 0.35"/>
     </joint>
     <!-- Camera -->
